File: analog-lorenz-attractor.kicad_sch (KiCad schematic)
At the start: 0 parts

Commit message: Draw schematic for equations circuits
Parts:
- added J1, J2, J3: Conn_Coaxial, symbol Connector:Conn_Coaxial
- added R10, R24, R26, R27, R28, R29, R31, R32, R33, R34, R36, R37, R38, R39, R41, R43, R44, R45, R46, R47, R48, R49: R_US, symbol Device:R_US
- added R11, R30, R35, R40, R42, R9: PT01-D115D-B104, 3_Potentiometer_THT:TRIM_PT01-D115D-B104, symbol 3_Potentiometer_THT:PT01-D115D-B104
- added U2, U7: AD633JNZ, 2_Amplifier_Multiplier:AD633JNZ, symbol 2_Amplifier_Multiplier:AD633JNZ
- added U4, U5, U6: ADA4096-2ACPZ-R7, 1_Amplifier_Operational:ADA4096-2ACPZ-R7, symbol 1_Amplifier_Operational:ADA4096-2ACPZ-R7
Connections:
- new net: R35.3, R38.1
- new net: R42.3, R46.1
- new net: R10.2, R24.1, U5.5 (INB+)
- new net: R30.3, R31.1
- new net: R26.1, R27.1, U6.5 (INB+)
- new net: R29.2, U6.6 (INB-)
- new net: R32.2, R34.2
- new net +15V: R11.2, R30.2, R35.2, R40.2, R42.2, R9.2, U2.8 (+VS), U4.8 (V+), U5.8 (V+), U6.8 (V+), U7.8 (+VS)
- new net -15V: U2.5 (-VS), U4.4 (V-), U5.4 (V-), U6.4 (V-), U7.5 (-VS)
- new net BETA: R48.2, R9.1, U6.2 (INA-)
- new net GND: J1.2 (Ext), J2.2 (Ext), J3.2 (Ext), R10.1, R26.2, R30.1, R33.1, R34.1, R35.1, R36.1, R37.1, R40.1, R41.1, R42.1, R45.1, R48.1, R49.1, U2.2 (X2), U2.4 (Y2), U2.6 (Z), U7.2 (X2), U7.4 (Y2), U7.6 (Z)
- new net RHO-Z: U2.3 (Y1), U5.1 (OUTA)
- new net RHO_RHO-Z: R31.2, R32.1, R33.2, U5.3 (INA+)
- new net SIGMA: R11.1, R49.2, U4.6 (INB-)
- new net SIGMA(Y-X): J1.1 (In), R11.3, U4.7 (OUTB)
- new net X(RHO-Z): R24.2, U2.7 (W)
- new net X(RHO-Z)-Y: J2.1 (In), U5.7 (OUTB)
- new net XY: R27.2, U7.7 (W)
- new net XY-ZBETA: J3.1 (In), R28.2, R29.1, U6.7 (OUTB)
- new net X_X(RHO-Z): R40.3, R43.1, U2.1 (X1)
- new net X_XY: R41.2, R43.2, R44.1, U7.1 (X1)
- new net X_Y-X: R44.2, U4.2 (INA-)
- new net Y-X: U4.1 (OUTA), U4.5 (INB+)
- new net Y/10: R36.2, R38.2, R39.1, U5.6 (INB-), U7.3 (Y1)
- new net Y_Y-X: R37.2, R39.2, U4.3 (INA+)
- new net ZBETA: R28.1, R9.3, U6.1 (OUTA)
- new net Z_RHO-Z: R47.2, U5.2 (INA-)
- new net Z_ZBETA: R45.2, R46.2, R47.1, U6.3 (INA+)
- no-connect marks 0 -> 3
Other:
- title: (none) -> Lorenz Equations

Commit message: Clear schematic for redesign
Parts:
- removed J1, J2, J3: Conn_Coaxial, symbol Connector:Conn_Coaxial
- removed R10, R24, R26, R27, R28, R29, R31, R32, R33, R34, R36, R37, R38, R39, R41, R43, R44, R45, R46, R47, R48, R49: R_US, symbol Device:R_US
- removed R11, R30, R35, R40, R42, R9: PT01-D115D-B104, 3_Potentiometer_THT:TRIM_PT01-D115D-B104, symbol 3_Potentiometer_THT:PT01-D115D-B104
- removed U2, U7: AD633JNZ, 2_Amplifier_Multiplier:AD633JNZ, symbol 2_Amplifier_Multiplier:AD633JNZ
- removed U4, U5, U6: ADA4096-2ACPZ-R7, 1_Amplifier_Operational:ADA4096-2ACPZ-R7, symbol 1_Amplifier_Operational:ADA4096-2ACPZ-R7
Connections:
- no-connect marks 3 -> 0
